File: Hardware/PCB2SCHEMATIC2/PCB2SCHEMATIC2/Schema_alimentation.kicad_pcb (KiCad board)
At the start: 2 copper layers, 48.3 x 48.3 mm, 19 parts, among them J1 Conn_02x07_Odd_Even, U1 STM32L412KBTx, U3 MPU-6050

Commit message: message
Routing:
- net GND: vias 1 -> 2
- net (no net): vias 113 -> 112
Other:
- board size 48.3 x 48.3 mm -> 110.2 x 48.3 mm
Changed lines of the file:
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@@
   (gr_line (start 155.01725 97.14) (end 155.01725 62.88)
+    (stroke (width 0.1) (type default)) (layer "Edge.Cuts"))
+  (gr_line (start 239.664 56.896) (end 258.176 56.896)
     (stroke (width 0.1) (type default)) (layer "Edge.Cuts"))
   (gr_line (start 203.27725 62.88) (end 203.27725 97.14)
@@
   (gr_arc (start 203.27725 97.14) (mid 201.226997 102.089747) (end 196.27725 104.14)
     (stroke (width 0.1) (type default)) (layer "Edge.Cuts"))
+  (gr_arc (start 258.176 56.896) (mid 263.125747 58.946253) (end 265.176 63.896)
+    (stroke (width 0.1) (type default)) (layer "Edge.Cuts"))
+  (gr_arc (start 232.664 63.896) (mid 234.714253 58.946253) (end 239.664 56.896)
+    (stroke (width 0.1) (type default)) (layer "Edge.Cuts"))
+  (gr_line (start 258.176 89.408) (end 239.664 89.408)
+    (stroke (width 0.1) (type default)) (layer "Edge.Cuts"))
   (gr_line (start 162.01725 55.88) (end 196.27725 55.88)
+    (stroke (width 0.1) (type default)) (layer "Edge.Cuts"))
+  (gr_line (start 265.176 63.896) (end 265.176 82.408)
+    (stroke (width 0.1) (type default)) (layer "Edge.Cuts"))
+  (gr_arc (start 239.664 89.408) (mid 234.714253 87.357747) (end 232.664 82.408)
     (stroke (width 0.1) (type default)) (layer "Edge.Cuts"))
   (gr_arc (start 196.27725 55.88) (mid 201.226997 57.930253) (end 203.27725 62.88)
     (stroke (width 0.1) (type default)) (layer "Edge.Cuts"))
+  (gr_line (start 232.664 82.408) (end 232.664 63.896)
+    (stroke (width 0.1) (type default)) (layer "Edge.Cuts"))
   (gr_arc (start 162.01725 104.14) (mid 157.067503 102.089747) (end 155.01725 97.14)
+    (stroke (width 0.1) (type default)) (layer "Edge.Cuts"))
+  (gr_arc (start 265.176 82.408) (mid 263.125747 87.357747) (end 258.176 89.408)
     (stroke (width 0.1) (type default)) (layer "Edge.Cuts"))
   (gr_text "T" (at 168.91 61.722) (layer "F.Cu")
@@
     (pts (xy 208.35725 55.88) (xy 208.35725 104.14))
     (height 58.42)
-    (gr_text "48,2600 mm" (at 148.13725 80.01 90) (layer "F.Cu")
+    (gr_text "48.2600 mm" (at 148.13725 80.01 90) (layer "F.Cu")
       (effects (font (size 1.5 1.5) (thickness 0.3)))
     )
@@
     (pts (xy 155.01725 109.22) (xy 203.27725 109.22))
     (height -58.42)
-    (gr_text "48,2600 mm" (at 179.14725 49) (layer "F.Cu")
+    (gr_text "48.2600 mm" (at 179.14725 49) (layer "F.Cu")
       (effects (font (size 1.5 1.5) (thickness 0.3)))
     )
@@
   (via (at 202.438 84.074) (size 0.8) (drill 0.4) (layers "F.Cu" "B.Cu") (net 0))
   (via (at 188.468 56.896) (size 0.8) (drill 0.4) (layers "F.Cu" "B.Cu") (net 0))
-  (via (at 155.956 96.52) (size 0.8) (drill 0.4) (layers "F.Cu" "B.Cu") (net 0))
   (via (at 155.956 64.516) (size 0.8) (drill 0.4) (layers "F.Cu" "B.Cu") (net 0))
   (via (at 166.624 103.378) (size 0.8) (drill 0.4) (layers "F.Cu" "B.Cu") (net 0))
@@
   (segment (start 197.866 75.692) (end 200.152 77.978) (width 0.3) (layer "B.Cu") (net 1))
   (segment (start 200.152 77.978) (end 200.152 82.211328) (width 0.3) (layer "B.Cu") (net 1))
+  (via (at 155.956 96.52) (size 0.8) (drill 0.4) (layers "F.Cu" "B.Cu") (free) (net 2))
   (via (at 155.956 98.044) (size 0.8) (drill 0.4) (layers "F.Cu" "B.Cu") (free) (net 2))
   (segment (start 185.264371 74.168) (end 185.808 74.168) (width 0.5) (layer "F.Cu") (net 3))
