File: Hardware/PCB2SCHEMATIC2/PCB2V1/PCBV1.kicad_sch (KiCad schematic)
At the start: 20 parts, among them J1 Conn_01x03, J2 Conn_01x08, J3 Conn_02x07_Odd_Even, J4 Conn_01x03, U1 STM32L412KBTx

Commit message: message
Parts:
- removed C5: 100n, Capacitor_SMD:C_0603_1608Metric_Pad1.08x0.95mm_HandSolder, symbol Device:C_Small
- removed J1, J4: Conn_01x03, Connector_JST:JST_XH_B3B-XH-A_1x03_P2.50mm_Vertical, symbol Connector_Generic:Conn_01x03
- removed J2: Conn_01x08, Connector_JST:JST_XH_B8B-XH-A_1x08_P2.50mm_Vertical, symbol Connector_Generic:Conn_01x08
- removed J3: Conn_02x07_Odd_Even, Connector_PinHeader_1.27mm:PinHeader_2x07_P1.27mm_Vertical_SMD, symbol Connector_Generic:Conn_02x07_Odd_Even
- added C2: 100n, Capacitor_SMD:C_0603_1608Metric_Pad1.08x0.95mm_HandSolder, symbol Device:C_Small
- added J1: Conn_02x07_Odd_Even, Connector_PinHeader_1.27mm:PinHeader_2x07_P1.27mm_Vertical_SMD, symbol Connector_Generic:Conn_02x07_Odd_Even
- added J2, J3: Conn_01x03, Connector_JST:JST_XH_B3B-XH-A_1x03_P2.50mm_Vertical, symbol Connector_Generic:Conn_01x03
- added J4: Conn_01x08, Connector_JST:JST_XH_B8B-XH-A_1x08_P2.50mm_Vertical, symbol Connector_Generic:Conn_01x08
- C1: value 100n -> 4u7
- C3: value 4u7 -> 100n
- R3: value 1k -> 100K
- R4: value 100K -> 1k
Connections:
- net +3.3V: now also C1.1, C2.1, J1.3 (Pin_3), J4.1 (Pin_1); no longer C4.1
- net BOUTON_RESET: now also C4.1, J1.12 (Pin_12); no longer C1.1
- net ESC1: now also J2.1 (Pin_1)
- net ESC2: now also J3.1 (Pin_1)
- net GND: now also C2.2, J1.11 (Pin_11), J1.5 (Pin_5), J1.7 (Pin_7), J2.3 (Pin_3), J3.3 (Pin_3), J4.2 (Pin_2)
- net SCL: now also J4.3 (Pin_3)
- net SDA: now also J4.4 (Pin_4)
- net SWDCK: now also J1.6 (Pin_6)
- net SWDIO: now also J1.4 (Pin_4)
- net USART2_RX: now also J1.13 (Pin_13)
- net USART2_TX: now also J1.14 (Pin_14)
- net at R4.1: now also D3.1 (K); no longer U1.30 (PB7)
- net at R3.1: now also U1.30 (PB7); no longer D3.1 (K)
Other:
- company: ENSEA -> (none)
- title: PROJET D'ELECTRONIQUE -> (none)
