File: Hardware/projet-pcbpuissance/projet-pcbpuissance.kicad_pcb (KiCad board)
At the start: 2 copper layers, 35 parts, among them J2 Conn_01x02, J3 Conn_01x02, J4 Conn_01x02, U1 MAX5033DUSA+, U2 MAX5033DUSA+

Commit message: Modif
Routing:
- net Batterie 11.1 V: track 104.1 -> 158.1 mm
- net GND: track 0.00 -> 5.48 mm, vias 0 -> 1
- added copper zone on B.Cu, net GND
- added copper zone on F.Cu, net GND
Other:
- board outline added: 83.8 x 61 mm
- board text added: "Hovercraft"
Changed lines of the file:
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@@
     )
+  )
+  (gr_line (start 171.0925 65.31) (end 171.0925 116.11)
+    (stroke (width 0.1) (type default)) (layer "Edge.Cuts"))
+  (gr_line (start 92.3525 60.23) (end 166.0125 60.23)
+    (stroke (width 0.1) (type default)) (layer "Edge.Cuts"))
+  (gr_arc (start 87.2725 65.31) (mid 88.760398 61.717898) (end 92.3525 60.23)
+    (stroke (width 0.1) (type default)) (layer "Edge.Cuts"))
+  (gr_line (start 87.2725 65.31) (end 87.2725 116.11)
+    (stroke (width 0.1) (type default)) (layer "Edge.Cuts"))
+  (gr_line (start 166.0125 121.19) (end 92.3525 121.19)
+    (stroke (width 0.1) (type default)) (layer "Edge.Cuts"))
+  (gr_arc (start 92.3525 121.19) (mid 88.760398 119.702102) (end 87.2725 116.11)
+    (stroke (width 0.1) (type default)) (layer "Edge.Cuts"))
+  (gr_arc (start 171.0925 116.11) (mid 169.604602 119.702102) (end 166.0125 121.19)
+    (stroke (width 0.1) (type default)) (layer "Edge.Cuts"))
+  (gr_arc (start 166.0125 60.23) (mid 169.604602 61.717898) (end 171.0925 65.31)
+    (stroke (width 0.1) (type default)) (layer "Edge.Cuts"))
+  (gr_text "Hovercraft\n" (at 105.0525 67.85) (layer "Dwgs.User")
+    (effects (font (size 1 1) (thickness 0.15)) (justify left bottom))
   )
   (segment (start 160.9325 100.87) (end 160.9325 87.99) (width 0.3) (layer "F.Cu") (net 1))
@@
   (segment (start 108.8625 92.3375) (end 108.8625 85.895) (width 0.3) (layer "F.Cu") (net 1))
   (segment (start 160.9325 87.99) (end 160.9325 75.47) (width 0.3) (layer "F.Cu") (net 1))
+  (segment (start 112.6725 108.33) (end 157.960978 108.33) (width 0.3) (layer "F.Cu") (net 1))
   (segment (start 113.9425 88.01) (end 160.9125 88.01) (width 0.3) (layer "F.Cu") (net 1))
   (segment (start 155.8475 72.93) (end 158.3925 72.93) (width 0.3) (layer "F.Cu") (net 1))
   (segment (start 106.1875 107.22) (end 107.5925 107.22) (width 0.3) (layer "F.Cu") (net 1))
+  (segment (start 160.9325 105.358478) (end 160.9325 100.87) (width 0.3) (layer "F.Cu") (net 1))
   (segment (start 111.5625 107.22) (end 112.6725 108.33) (width 0.3) (layer "F.Cu") (net 1))
+  (segment (start 157.960978 108.33) (end 160.9325 105.358478) (width 0.3) (layer "F.Cu") (net 1))
+  (segment (start 98.2475 108.49) (end 97.4325 107.675) (width 0.3) (layer "F.Cu") (net 2))
+  (segment (start 101.7575 87.165) (end 99.9725 87.165) (width 0.3) (layer "F.Cu") (net 2))
+  (segment (start 100.7875 108.49) (end 98.2475 108.49) (width 0.3) (layer "F.Cu") (net 2))
+  (via (at 99.9725 87.165) (size 0.8) (drill 0.4) (layers "F.Cu" "B.Cu") (free) (net 2))
   (segment (start 101.7575 85.895) (end 99.83 85.895) (width 0.3) (layer "F.Cu") (net 3))
   (segment (start 99.83 85.895) (end 98.7025 84.7675) (width 0.3) (layer "F.Cu") (net 3))
@@
   (segment (start 107.0425 84.625) (end 105.5075 83.09) (width 0.3) (layer "F.Cu") (net 17))
   (segment (start 105.5075 83.09) (end 102.9675 80.55) (width 0.3) (layer "F.Cu") (net 17))
+  (zone (net 2) (net_name "GND") (layer "F.Cu") (hatch edge 0.5)
+    (connect_pads (clearance 0.5))
+    (min_thickness 0.25) (filled_areas_thickness no)
+    (fill yes (thermal_gap 0.5) (thermal_bridge_width 0.5))
+    (polygon
+      (pts
+        (xy 79.6525 52.61)
+        (xy 79.6525 126.27)
+        (xy 181.2525 126.27)
+        (xy 181.2525 52.61)
+      )
+    )
+  )
+  (zone (net 2) (net_name "GND") (layer "B.Cu") (hatch edge 0.5)
+    (priority 1)
+    (connect_pads (clearance 0.5))
+    (min_thickness 0.25) (filled_areas_thickness no)
+    (fill yes (thermal_gap 0.5) (thermal_bridge_width 0.5))
+    (polygon
+      (pts
+        (xy 79.6525 52.61)
+        (xy 79.6525 126.27)
+        (xy 181.2525 126.27)
+        (xy 181.2525 52.61)
+      )
+    )
+  )
 )

Commit message: Modif pcb puissance
Parts:
- moved J4 38.9 mm to (122.8, 108.5)
- moved J3 34.7 mm to (133.0, 108.5)
- moved J2 16.2 mm to (148.3, 85.6)
- moved H2 16.1 mm to (150.8, 111.0)
- moved H1 15.5 mm to (150.8, 67.8)
- moved R9 7.94 mm to (148.8, 80.5)
- moved D4 7.94 mm to (152.7, 80.5)
- moved R10 6.35 mm to (98.3, 94.5)
- moved R11 6.35 mm to (93.3, 103.4)
- moved U2 6.35 mm to (103.5, 101.5)
- moved C5 6.35 mm to (112.7, 104.7)
- moved C6 6.35 mm to (97.4, 100.5)
- moved C7 6.35 mm to (104.2, 97.1)
- moved R7 6.35 mm to (107.6, 106.3)
- moved R8 6.35 mm to (105.1, 107.2)
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Routing:
- net Batterie 11.1 V: track 158.1 -> 124.2 mm
- net Net-(U2-ON/~{OFF}): track 6.29 -> 5.00 mm
- net Net-(D2-K): track 32.4 -> 33.2 mm
Other:
- board size 83.8 x 61 mm -> 66 x 53.3 mm

Commit message: Modif pcb
Parts:
- moved R9 18.1 mm to (153.3, 98.1), turned to -90 degrees
- moved D4 13.6 mm to (153.3, 94.1), turned to 90 degrees
- moved D1 5.35 mm to (141.5, 70.4)
- moved R3 5.35 mm to (136.4, 70.4)
- moved C4 5.08 mm to (145.2, 80.5)
- moved H1 5.08 mm to (150.8, 72.9)
- moved H3 5.08 mm to (94.9, 72.9)
- moved J2 2.54 mm to (148.2, 88.2)
- moved H2 2.54 mm to (150.8, 108.5)
- moved H4 2.54 mm to (94.9, 108.5)
Routing:
- net Batterie 11.1 V: track 124.2 -> 122.5 mm
- net +3.3V: track 14.6 -> 15.8 mm
Other:
- board size 66 x 53.3 mm -> 66 x 45.7 mm

Commit message: Modif(en cours)
Parts:
- D2, D6: footprint Diode_THT:D_DO-201AD_P12.70mm_Horizontal -> Diode_SMD:D_SMA_Handsoldering
- moved R11 8.24 mm to (101.3, 105.1), turned to 180 degrees
- moved R5 8.11 mm to (102.0, 87.5), turned to 180 degrees
- moved R10 6.82 mm to (97.4, 101.3), turned to 90 degrees
- moved R4 6.51 mm to (98.0, 84.2), turned to -90 degrees
- moved C8 2.51 mm to (143.2, 96.3)
- moved R1 2.37 mm to (108.3, 88.3)
- moved C6 1.83 mm to (99.0, 101.4)
- moved C2 1.76 mm to (99.6, 84.3)
- moved R2 1.61 mm to (106.8, 88.4)
- moved R8 1.30 mm to (104.9, 105.9)
- moved R7 1.22 mm to (106.4, 106.0)
- moved C1 1.01 mm to (114.4, 87.7)
Routing:
- net GND: track 5.48 -> 1.87 mm, vias 1 -> 4
- net Net-(U2-VD): track 3.88 -> 1.93 mm
- net Net-(U1-VD): track 3.52 -> 1.88 mm
- net Net-(D2-K): track 33.2 -> 31.9 mm

Commit message: Modif PCB
Parts:
- R1, R7: value R_Small -> 1M
- R2, R8: value R_Small -> 390K
- moved D6 11.8 mm to (110.7, 79.4)
- moved D1 11.7 mm to (129.8, 70.0)
- moved R3 11.7 mm to (124.7, 70.0)
- moved C4 11.4 mm to (134.3, 77.6)
- moved D4 10.2 mm to (143.5, 91.6)
- moved R9 10.2 mm to (143.5, 95.6)
- moved L1 9.91 mm to (122.7, 77.4)
- moved R6 9.28 mm to (122.8, 87.8)
- moved D2 9.28 mm to (112.3, 94.8)
- moved D3 9.28 mm to (128.0, 87.8)
- moved H1 7.96 mm to (142.8, 73.0)
- moved H2 7.96 mm to (142.8, 108.5)
- moved L2 7.72 mm to (124.0, 95.2)
- moved C8 7.66 mm to (135.6, 95.0)
- moved H3 5.59 mm to (100.5, 72.7)
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Routing:
- net Batterie 11.1 V: track 122.5 -> 111.0 mm, vias 0 -> 2
- net Net-(U2-FB): track 16.8 -> 5.74 mm
- net Net-(U1-FB): track 15.7 -> 5.58 mm
- net Net-(D6-K): track 30.2 -> 24.8 mm
- net Net-(D2-K): track 31.9 -> 27.4 mm
- net +3.3V: track 15.8 -> 11.6 mm
- net Net-(D3-K): track 3.33 -> 0.00 mm
- net Net-(U1-ON/~{OFF}): track 7.13 -> 4.00 mm
- net 7.4V: track 15.1 -> 13.1 mm
- net GND: track 1.87 -> 3.85 mm
Other:
- board size 66 x 45.7 mm -> 52.4 x 45.8 mm
