File: Hardware/projet-pcbpuissance/projet-pcbpuissance.kicad_sch (KiCad schematic)
At the start: 32 parts, among them U1 MAX5033DUSA+, U2 MAX5033DUSA+

Commit message: Modification pcb-puissance
Parts:
- removed C1, C5: 47µF, Capacitor_SMD:C_0603_1608Metric_Pad1.08x0.95mm_HandSolder, symbol Device:C_Small
- added C1, C5: 47µF, Capacitor_SMD:C_0603_1608Metric_Pad1.08x0.95mm_HandSolder, symbol Device:C_Polarized_Small
- added J1: Conn_01x08, Connector_JST:JST_XH_B8B-XH-AM_1x08_P2.50mm_Vertical, symbol Connector_Generic:Conn_01x08
- added J2, J3, J4: Conn_01x02, Connector_JST:JST_XH_B2B-XH-AM_1x02_P2.50mm_Vertical, symbol Connector_Generic:Conn_01x02
- added J5, J6: Conn_01x03, Connector_JST:JST_XH_B3B-XH-AM_1x03_P2.50mm_Vertical, symbol Connector_Generic:Conn_01x03
- R3: renamed from R9; value R_Small -> 1k
- R6: renamed from R10; value R_Small -> 1k
- R9: renamed from R11; value R_Small -> 1k
- renumbered D3 to D1, D1 to D2, D4 to D3, D5 to D4, D2 to D5, R2 to R1, R7 to R10, R8 to R11, R1 to R2, R3 to R4, R4 to R5, R5 to R7, R6 to R8
Connections:
- net Batterie 11.1 V: now also C1.1, C5.1
- net GND: now also C1.2, C5.2, J2.2 (Pin_2), J3.2 (Pin_2), J4.2 (Pin_2), J5.3 (Pin_3), J6.3 (Pin_3)
- new net VCC: J2.1 (Pin_1), J3.1 (Pin_1), J4.1 (Pin_1)
Other:
- note added: "PWM (motor control) x2"

Commit message: Modif
Connections:
- net +3.3V: now also J1.1 (Pin_1)
- net GND: now also J1.8 (Pin_8)
- net SCL: now also J1.3 (Pin_3)
- net SDA: now also J1.5 (Pin_5)
Changed lines of the file:
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@@
+    (stroke (width 0) (type default))
+  )
+  (wire (pts (xy 163.83 52.07) (xy 163.83 54.61))
     (stroke (width 0) (type default))
   )
@@
     (stroke (width 0) (type default))
   )
+  (wire (pts (xy 177.8 52.07) (xy 163.83 52.07))
+    (stroke (width 0) (type default))
+  )
   (wire (pts (xy 55.88 62.23) (xy 55.88 63.5))
     (stroke (width 0) (type default))
@@
     (stroke (width 0) (type default))
   )
+  (wire (pts (xy 163.83 34.29) (xy 163.83 33.02))
+    (stroke (width 0) (type default))
+  )
   (wire (pts (xy 170.18 71.12) (xy 181.61 71.12))
     (stroke (width 0) (type default))
@@
     (stroke (width 0) (type default))
   )
+  (wire (pts (xy 177.8 34.29) (xy 163.83 34.29))
+    (stroke (width 0) (type default))
+  )
   (wire (pts (xy 262.89 86.36) (xy 247.65 86.36))
     (stroke (width 0) (type default))
@@
     (stroke (width 0) (type default))
   )
+  (wire (pts (xy 166.37 39.37) (xy 177.8 39.37))
+    (stroke (width 0) (type default))
+  )
   (wire (pts (xy 43.18 83.82) (xy 43.18 81.28))
     (stroke (width 0) (type default))
@@
   )
   (wire (pts (xy 259.08 41.91) (xy 254 41.91))
+    (stroke (width 0) (type default))
+  )
+  (wire (pts (xy 166.37 44.45) (xy 177.8 44.45))
     (stroke (width 0) (type default))
   )
@@
     )
   )
-  (global_label "SCL" (shape input) (at 162.56 39.37 0) (fields_autoplaced)
-    (effects (font (size 1.27 1.27)) (justify left))
-    (property "Intersheetrefs" "${INTERSHEET_REFS}" (at 168.9734 39.37 0)
-      (effects (font (size 1.27 1.27)) (justify left) hide)
+  (global_label "SCL" (shape input) (at 166.37 39.37 180) (fields_autoplaced)
+    (effects (font (size 1.27 1.27)) (justify right))
+    (property "Intersheetrefs" "${INTERSHEET_REFS}" (at 159.9566 39.37 0)
+      (effects (font (size 1.27 1.27)) (justify right) hide)
     )
   )
@@
     )
   )
-  (global_label "SDA" (shape input) (at 163.83 44.45 0) (fields_autoplaced)
-    (effects (font (size 1.27 1.27)) (justify left))
-    (property "Intersheetrefs" "${INTERSHEET_REFS}" (at 170.3039 44.45 0)
-      (effects (font (size 1.27 1.27)) (justify left) hide)
+  (global_label "SDA" (shape input) (at 166.37 44.45 180) (fields_autoplaced)
+    (effects (font (size 1.27 1.27)) (justify right))
+    (property "Intersheetrefs" "${INTERSHEET_REFS}" (at 159.8961 44.45 0)
+      (effects (font (size 1.27 1.27)) (justify right) hide)
     )
   )
@@
     )
   )
-  (symbol (lib_id "power:GND") (at 163.83 49.53 0) (unit 1)
-    (in_bom yes) (on_board yes) (dnp no) (fields_autoplaced)
-    (property "Reference" "#PWR016" (at 163.83 55.88 0)
-      (effects (font (size 1.27 1.27)) hide)
-    )
-    (property "Value" "GND" (at 163.83 54.61 0)
-      (effects (font (size 1.27 1.27)))
-    )
-    (property "Footprint" "" (at 163.83 49.53 0)
-      (effects (font (size 1.27 1.27)) hide)
-    )
-    (property "Datasheet" "" (at 163.83 49.53 0)
-      (effects (font (size 1.27 1.27)) hide)
-    )
+  (symbol (lib_id "power:GND") (at 163.83 54.61 0) (unit 1)
+    (in_bom yes) (on_board yes) (dnp no) (fields_autoplaced)
+    (property "Reference" "#PWR016" (at 163.83 60.96 0)
+      (effects (font (size 1.27 1.27)) hide)
+    )
+    (property "Value" "GND" (at 163.83 59.69 0)
+      (effects (font (size 1.27 1.27)))
+    )
+    (property "Footprint" "" (at 163.83 54.61 0)
+      (effects (font (size 1.27 1.27)) hide)
+    )
+    (property "Datasheet" "" (at 163.83 54.61 0)
+      (effects (font (size 1.27 1.27)) hide)
+    )

Commit message: Modification pcb puissance
Parts:
- removed J1: Conn_01x08, Connector_JST:JST_XH_B8B-XH-AM_1x08_P2.50mm_Vertical, symbol Connector_Generic:Conn_01x08
- removed J5, J6: Conn_01x03, Connector_JST:JST_XH_B3B-XH-AM_1x03_P2.50mm_Vertical, symbol Connector_Generic:Conn_01x03
Other:
- note added: "Connecteurs"
- note removed: "Connecteurs ?"
- note removed: "PWM (motor control) x2"
- moved on the sheet: J2, J3, J4

Commit message: Modif
Parts:
- removed D2, D5: D_Zener, Diode_SMD:Littelfuse_PolyZen-LS, symbol Device:D_Zener
- added D2, D6: D_Schottky, Diode_THT:D_DO-201AD_P12.70mm_Horizontal, symbol Device:D_Schottky
- C1, C4, C5, C8: footprint Capacitor_SMD:C_0603_1608Metric_Pad1.08x0.95mm_HandSolder -> Capacitor_SMD:CP_Elec_6.3x7.7
- L1, L2: footprint Inductor_SMD:L_0805_2012Metric_Pad1.05x1.20mm_HandSolder -> Inductor_SMD:L_12x12mm_H6mm
Connections:
- net GND: now also D2.2 (A), D6.2 (A)
- net at C3.1, L1.1, R4.2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: now also D6.1 (K)
- net at C7.1, L2.1, R10.2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: now also D2.1 (K)

Commit message: Modif
Connections:
- net VCC is gone; now on net Batterie 11.1 V: J2.1 (Pin_1), J3.1 (Pin_1), J4.1 (Pin_1)
Changed lines of the file:
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@@
+    (stroke (width 0) (type default))
+  )
+  (wire (pts (xy 21.59 29.21) (xy 21.59 30.48))
     (stroke (width 0) (type default))
   )
@@
   )
   (wire (pts (xy 167.64 71.12) (xy 170.18 71.12))
-    (stroke (width 0) (type default))
-  )
-  (wire (pts (xy 21.59 30.48) (xy 21.59 27.94))
     (stroke (width 0) (type default))
   )
@@
     )
   )
+  (global_label "Batterie 11.1 V" (shape input) (at 21.59 29.21 90) (fields_autoplaced)
+    (effects (font (size 1.27 1.27)) (justify left))
+    (property "Intersheetrefs" "${INTERSHEET_REFS}" (at 21.59 11.6085 90)
+      (effects (font (size 1.27 1.27)) (justify left) hide)
+    )
+  )
   (global_label "Batterie 11.1 V" (shape input) (at 43.18 54.61 180) (fields_autoplaced)
     (effects (font (size 1.27 1.27)) (justify right))
@@
         )
       )
-    )
-  )
-  (symbol (lib_id "power:VCC") (at 21.59 27.94 0) (unit 1)
-    (in_bom yes) (on_board yes) (dnp no) (fields_autoplaced)
-    (property "Reference" "#PWR022" (at 21.59 31.75 0)
-      (effects (font (size 1.27 1.27)) hide)
-    )
-    (property "Value" "VCC" (at 21.59 24.13 0)
-      (effects (font (size 1.27 1.27)))
-    )
-    (property "Footprint" "" (at 21.59 27.94 0)
-      (effects (font (size 1.27 1.27)) hide)
-    )
-    (property "Datasheet" "" (at 21.59 27.94 0)
-      (effects (font (size 1.27 1.27)) hide)
-    )
-    (pin "1")
-    (instances
-      (project "projet-pcbpuissance"
-        (path "/2869d089-2104-43b1-9a93-26592258e38f"
-          (reference "#PWR022") (unit 1)
-        )
-      )
-      (project "Schema_alimentation"
-        (path "/6a1fa79b-29e8-4816-8d7e-fabfcde671cf"
-          (reference "#PWR012") (unit 1)
-        )
-      )

Commit message: Modif
Connections:
- net 11.1V is gone; now on net Batterie 11.1 V: D4.2 (A)
Changed lines of the file:
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@@
-    )
-  )
-  (global_label "11.1V" (shape input) (at 161.29 130.81 0) (fields_autoplaced)
-    (effects (font (size 1.27 1.27)) (justify left))
-    (property "Intersheetrefs" "${INTERSHEET_REFS}" (at 169.5177 130.81 0)
-      (effects (font (size 1.27 1.27)) (justify left) hide)
     )
   )
@@
       (effects (font (size 1.27 1.27)) (justify left) hide)
     )
+  )
+  (global_label "Batterie 11.1 V" (shape input) (at 161.29 130.81 0) (fields_autoplaced)
+    (effects (font (size 1.27 1.27)) (justify left))
+    (property "Intersheetrefs" "${INTERSHEET_REFS}" (at 178.8915 130.81 0)
+      (effects (font (size 1.27 1.27)) (justify left) hide)
+    )

Commit message: Modif(en cours)
Parts:
- D2, D6: footprint Diode_THT:D_DO-201AD_P12.70mm_Horizontal -> Diode_SMD:D_SMA_Handsoldering
Changed lines of the file:
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@@
       (effects (font (size 1.27 1.27)) (justify left))
     )
-    (property "Footprint" "Diode_THT:D_DO-201AD_P12.70mm_Horizontal" (at 181.61 74.93 0)
+    (property "Footprint" "Diode_SMD:D_SMA_Handsoldering" (at 181.61 74.93 0)
       (effects (font (size 1.27 1.27)) hide)
     )
@@
       (effects (font (size 1.27 1.27)) (justify left))
     )
-    (property "Footprint" "Diode_THT:D_DO-201AD_P12.70mm_Horizontal" (at 87.63 74.93 0)
-      (effects (font (size 1.27 1.27)) hide)
-    )
+    (property "Footprint" "Diode_SMD:D_SMA_Handsoldering" (at 87.63 74.93 0)
+      (effects (font (size 1.27 1.27)) hide)
+    )

Commit message: Modif PCB
Parts:
- R1, R7: value R_Small -> 1M
- R2, R8: value R_Small -> 390K
Changed lines of the file:
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@@
       (effects (font (size 1.27 1.27)) (justify left))
     )
-    (property "Value" "R_Small" (at 139.7 65.405 0)
+    (property "Value" "1M" (at 139.7 65.405 0)
       (effects (font (size 1.27 1.27)) (justify left))
     )
@@
       (effects (font (size 1.27 1.27)) (justify left))
     )
-    (property "Value" "R_Small" (at 45.72 65.405 0)
+    (property "Value" "1M" (at 45.72 65.405 0)
       (effects (font (size 1.27 1.27)) (justify left))
     )
@@
       (effects (font (size 1.27 1.27)) (justify left))
     )
-    (property "Value" "R_Small" (at 139.7 80.645 0)
+    (property "Value" "390K" (at 139.7 80.645 0)
       (effects (font (size 1.27 1.27)) (justify left))
     )
@@
       (effects (font (size 1.27 1.27)) (justify left))
     )
-    (property "Value" "R_Small" (at 45.72 80.645 0)
-      (effects (font (size 1.27 1.27)) (justify left))
-    )
+    (property "Value" "390K" (at 45.72 80.645 0)
+      (effects (font (size 1.27 1.27)) (justify left))
+    )
