File: Hardware/PCB2V1/PCBV1.kicad_pcb (KiCad board)
At the start: 2 copper layers, 38 x 40 mm, 21 parts, among them J1 Conn_02x07_Odd_Even, J2 Conn_01x03, J3 Conn_01x03, J4 Conn_01x08, SW1 SW_Push, U1 STM32L412KBTx

Commit message: message
Parts:
- removed D3: LED_Small, LED_SMD:LED_0603_1608Metric_Pad1.05x0.95mm_HandSolder
- removed R4: 1k, Resistor_SMD:R_0603_1608Metric_Pad0.98x0.95mm_HandSolder
- added J5: Conn_01x02, Connector_JST:JST_XH_B2B-XH-A_1x02_P2.50mm_Vertical, F.Cu at (137.2, 134.8)
- moved C3 12.9 mm to (139.8, 122.5)
- moved C2 11.0 mm to (138.8, 125.0), turned to -90 degrees
- moved C1 9.75 mm to (137.2, 125.0), turned to -90 degrees
- moved J2 3.51 mm to (146.0, 134.8)
- moved D1 1.40 mm to (140.8, 119.7)
- moved D2 1.40 mm to (140.8, 116.1)
- moved R1 1.40 mm to (142.2, 119.7)
- moved R2 1.40 mm to (142.2, 116.1)
- moved R3 0.71 mm to (129.8, 113.5)
- moved J1 0.70 mm to (147.7, 119.7)
- moved J3 0.50 mm to (141.8, 105.0)
Connections:
- U1 pad 13: SCL -> unconnected-(U1-PA7-Pad13)
- U1 pad 19: LED_USER2 -> SCL
Routing:
- net GND: track 120.1 -> 25.8 mm, vias 5 -> 2
- net +3.3V: track 68.5 -> 102.5 mm
- net BOUTON_RESET: track 29.1 -> 48.9 mm
- net SDA: track 19.5 -> 29.8 mm
- net SWDIO: track 16.3 -> 21.4 mm
- net SCL: track 25.3 -> 30.1 mm, vias 0 -> 2
- net USART2_RX: track 18.6 -> 22.9 mm
- net ESC1: track 16.0 -> 20.1 mm, vias 2 -> 0
- net SWDCK: track 22.1 -> 26.1 mm
- net LED_USER2: track 3.65 -> 0.00 mm
- net USART2_TX: track 36.1 -> 33.9 mm
- net Net-(D3-K): track 1.57 -> 0.00 mm
- net LED_USER1: track 2.99 -> 4.50 mm
- net LED_PWR: track 2.59 -> 4.07 mm
- net BOUTON_USR: track 25.9 -> 26.8 mm
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